Commit message: Complete Step 2

File: Step2/rrbot_on_table.urdf.xacro (robot description, xacro)
@@ -6,5 +6,5 @@
     <link name="world" />
     <xacro:table prefix="table_" parent="world">
-        <origin xyz="0 0 1" rpy="0 0 0" />
+        <origin xyz="0 0 0" rpy="0 0 0" />
     </xacro:table>
     <xacro:rrbot prefix="rrbot_" parent="table_top">

File: Step2/table_on_rrbot.urdf.xacro (robot description, xacro)
@@ -9,5 +9,5 @@
     </xacro:rrbot>
     <xacro:table prefix="table_" parent="rrbot_tool0">
-        <origin xyz="0 0 0" rpy="${pi} 0 0" />
+        <origin xyz="0 0 1" rpy="${pi} 0 0" />
     </xacro:table>
 </robot>
