Commit message: Complete Step 4

File: ws2/src/ur3e_on_table/urdf/ur3e_on_table.urdf.xacro (robot description, xacro)
@@ -5,5 +5,5 @@
     <link name="world" />
     <xacro:table prefix="table_" parent="world">
-        <origin xyz="0 0 1" rpy="0 0 0" />
+        <origin xyz="0 0 0" rpy="0 0 0" />
     </xacro:table>
     <!-- robot name parameter -->
